File: Faradometer.kicad_pcb (KiCad board)
At the start: 2 copper layers, 17 parts, among them J1 Screw_Terminal_01x06, U1 TL072CP, U2 TL072CP

Commit message: Describe what you changed
Parts:
- removed C1: 1n, Capacitor_SMD:C_0805_2012Metric
- removed J1: Screw_Terminal_01x06, Screw Terminal x6:TE_282836-6
- added H1: MountingHole_Pad, MountingHole:MountingHole_3.2mm_M3_DIN965_Pad, F.Cu at (136.4, 77.0)
- added H2: MountingHole_Pad, MountingHole:MountingHole_3.2mm_M3_DIN965_Pad, F.Cu at (155.8, 76.8)
- added J3: Conn_01x02_Pin, Connector_Molex:Molex_Nano-Fit_105313-xx02_1x02_P2.50mm_Horizontal, F.Cu at (137.7, 89.5)
- added J4: Conn_01x03_Pin, Connector_Molex:Molex_Nano-Fit_105313-xx03_1x03_P2.50mm_Horizontal, F.Cu at (156.8, 89.5)
- C2, C3: footprint Capacitor_SMD:C_0805_2012Metric -> Capacitor_SMD:C_0402_1005Metric_Pad0.74x0.62mm_HandSolder
- C5: footprint Capacitor_SMD:C_0805_2012Metric -> Capacitor_SMD:C_0603_1608Metric_Pad1.08x0.95mm_HandSolder
- C6: footprint Capacitor_SMD:C_0805_2012Metric -> Capacitor_SMD:C_0805_2012Metric_Pad1.18x1.45mm_HandSolder
- moved D1 44.5 mm to (158.2, 86.5), turned to 180 degrees
- moved C3 41.3 mm to (156.7, 83.4), turned to -90 degrees
- moved C2 39.9 mm to (138.8, 83.8), turned to 180 degrees
- moved R6 39.0 mm to (155.0, 82.8), turned to 90 degrees
- moved R7 38.8 mm to (138.9, 86.2), turned to -90 degrees
- moved R8 38.4 mm to (138.8, 81.6), turned to -90 degrees
- moved C5 37.2 mm to (136.9, 82.0), turned to -90 degrees
- moved U2 37.1 mm to (140.9, 86.1)
- moved U1 37.0 mm to (140.9, 75.3)
- moved R1 36.5 mm to (137.0, 86.1), turned to 90 degrees
- moved R3 35.8 mm to (151.2, 84.3)
- moved R2 34.9 mm to (135.0, 82.0), turned to 90 degrees
- moved C6 34.8 mm to (134.8, 85.9), turned to 90 degrees
- moved R5 34.2 mm to (151.2, 80.4), turned to 0 degrees
- moved R4 31.5 mm to (151.2, 82.4), turned to 0 degrees
Routing:
- net /VREF: track 87.1 -> 35.2 mm, vias 0 -> 4
- net +12V: track 85.0 -> 36.7 mm, vias 1 -> 3
- net /U2 1 IN -: track 40.0 -> 13.1 mm, vias 1 -> 0
- net /U2 2 IN -: track 30.0 -> 19.6 mm, vias 2 -> 0
- net /2 IN +: track 10.6 -> 3.86 mm
- net /2 IN -: track 5.84 -> 1.74 mm
- net /U2 2 out: track 5.10 -> 3.57 mm
- net /1 IN +: track 8.86 -> 9.77 mm
- net /U2 1 out: track 16.1 -> 16.6 mm, vias 0 -> 1
- net /2 out: track 27.9 -> 27.7 mm, vias 2 -> 0
Other:
- board outline added: 26.3 x 21.7 mm

Commit message: annotated schematic
Parts:
- removed U1, U2: TL072CP, TL072CP:P8
- added C104: 1n, Capacitor_SMD:C_0402_1005Metric_Pad0.74x0.62mm_HandSolder, F.Cu at (151.5, 77.2)
- added U101: TL072CP, Package_DIP:DIP-8_W7.62mm, F.Cu at (140.9, 75.4)
- added U102: TL072CP, Package_DIP:DIP-8_W7.62mm, F.Cu at (141.0, 86.1)
- moved J102 0.19 mm to (156.9, 89.4)
- moved R106 0.11 mm to (151.3, 82.3)
- moved R105 0.10 mm to (151.3, 84.3)
- moved R107 0.10 mm to (151.3, 80.4)
- renumbered C5 to C101, C2 to C102, C6 to C103, C3 to C105, D1 to D101, H2 to H101, H1 to H102, J3 to J101, J4 to J102, R1 to R101, R2 to R102, R7 to R103, R8 to R104, R3 to R105, R4 to R106, R5 to R107, R6 to R108
Connections:
- net /1 IN + renamed Net-(U101B-+)
- net /2 IN + renamed Net-(U101C-+)
- net /2 out renamed /SQ Out
- net /U2 1 IN - renamed /capacitor1
- net /U2 2 IN - renamed /V Out
- D101 pad 2: /U2 2 out -> Net-(D101-A)
- R104 pad 1: /1 IN - -> Net-(U101B--)
- R107 pad 1: /2 IN - -> Net-(U101C--)
Routing:
- net Net-(U101B--): track 0.00 -> 6.22 mm
- net /1 IN -: track 6.22 -> 0.00 mm
- net Net-(D101-A): track 0.00 -> 3.57 mm
- net /U2 2 out: track 3.57 -> 0.00 mm
- net Net-(U101C--): track 0.00 -> 1.74 mm
- net /2 IN -: track 1.74 -> 0.00 mm
- added copper zone on B.Cu, net GND
