File: _autosave-Faradometer.kicad_pcb (KiCad board)
At the start: 2 copper layers, 26 x 22.2 mm, 20 parts, among them J101 Conn_01x02_Pin, J102 Conn_01x03_Pin, U101 TL072CP, U102 TL072CP

Commit message: pcb change according to document
Parts:
- added C1: 100nF, Capacitor_SMD:C_0402_1005Metric_Pad0.74x0.62mm_HandSolder, F.Cu at (141.8, 64.8)
- added C2: 100nF, Capacitor_SMD:C_0402_1005Metric_Pad0.74x0.62mm_HandSolder, F.Cu at (141.8, 65.8)
- moved C101 0.35 mm to (130.0, 71.0)
Connections:
- net /U2 1 out renamed Net-(U102C-+)
Routing:
- net GND: vias 0 -> 2
Other:
- board size 26 x 22.2 mm -> 26 x 22 mm
